File: Lab8/kicad/kicad.kicad_pcb (KiCad board)
At the start: 32 copper layers, 146 x 91.4 mm, 20 parts, among them U1 OPB745, U2 TLC277, U3 TLC277

Commit message: near checkoff
Parts:
- removed U3: TLC277, TLC277CP:DIP794W45P254L959H508Q8
- 1k2, R8: moved to F.Cu
- C2, R5, R6, r4: moved to B.Cu
- U1: footprint Connector_PinSocket_2.54mm:PinSocket_1x08_P2.54mm_Vertical -> Connector_PinHeader_2.54mm:PinHeader_1x04_P2.54mm_Vertical
- moved OUT1 35.3 mm to (243.8, 106.7), turned to 0 degrees
- moved 1k2 35.1 mm to (203.2, 116.8), turned to 270 degrees
- moved R6 31.8 mm to (185.1, 94.0)
- moved R9 30.5 mm to (219.7, 108.0)
- moved R8 27.7 mm to (207.3, 110.5), turned to 0 degrees
- moved Vin2 25.0 mm to (232.4, 90.2)
- moved C2 24.2 mm to (201.9, 97.8), turned to 270 degrees
- moved D1 20.1 mm to (232.4, 101.6), turned to 270 degrees
- moved r4 18.8 mm to (172.7, 108.0), turned to 180 degrees
- moved R5 17.3 mm to (175.3, 101.6), turned to 180 degrees
- moved D2 17.3 mm to (236.2, 118.1), turned to 270 degrees
- moved C1 14.1 mm to (167.6, 101.6), turned to 180 degrees
- moved R3 13.0 mm to (168.9, 114.3), turned to 90 degrees
- moved U2 5.08 mm to (185.4, 108.0), turned to 0 degrees
- moved R1 1.27 mm to (153.7, 100.3), turned to 180 degrees
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Connections:
- U2 pad 5: (no net) -> Net-(C2-Pad1)
- U2 pad 6: (no net) -> Net-(1k2-Pad1)
- U2 pad 7: (no net) -> Net-(R8-Pad1)
Routing:
- net Net-(R5-Pad1): track 135.5 -> 18.2 mm
- net Net-(1k2-Pad2): track 176.3 -> 257.0 mm
- net Net-(C1-Pad2): track 39.8 -> 22.9 mm
- net Net-(R8-Pad1): track 34.8 -> 49.7 mm
- net Net-(C2-Pad1): track 30.0 -> 38.6 mm
- net Net-(R5-Pad2): track 7.38 -> 15.9 mm
- net Net-(C1-Pad1): track 19.9 -> 26.7 mm
- net Net-(D1-Pad2): track 34.2 -> 39.9 mm
- net Net-(D1-Pad1): track 6.48 -> 11.1 mm
- net Net-(R1-Pad2): track 7.51 -> 6.53 mm

Commit message: pcb done
Parts:
- R1, R2, R3, R5, R6, R8, R9, r4: footprint Resistor_SMD:R_0201_0603Metric -> Resistor_SMD:R_0201_0603Metric_Pad0.64x0.40mm_HandSolder
Routing:
- net Net-(R5-Pad1): track 18.2 -> 17.4 mm
Other:
- net class Default: clearance 0.2 -> 0.1
- rule trace_clearance: 0.2 -> 0.1
