File: Lab8/kicad/kicad.kicad_pcb (KiCad board)
At the start: 32 copper layers, 146 x 91.4 mm, 19 parts, among them U1 OPB745, U2 TLC277

Commit message: fixed some stuff
Parts:
- added GND2: GND, Connector_PinHeader_2.54mm:PinHeader_1x01_P2.54mm_Horizontal, F.Cu at (238.8, 138.4)
- 1k2, R1, R2, R3, R5, R6, R8, R9, r4: footprint Resistor_SMD:R_0201_0603Metric -> Resistor_THT:R_Axial_DIN0204_L3.6mm_D1.6mm_P1.90mm_Vertical
- C1: footprint Capacitor_SMD:CP_Elec_3x5.4 -> Capacitor_THT:CP_Radial_D4.0mm_P1.50mm
- C2: footprint Capacitor_SMD:CP_Elec_4x3 -> Capacitor_THT:CP_Radial_D4.0mm_P1.50mm
- D1, D2: footprint Diode_SMD:D_0201_0603Metric -> Capacitor_THT:CP_Axial_L10.0mm_D4.5mm_P15.00mm_Horizontal
- GND1: renamed from gnd1; value Conn_01x01_Male -> GND
- Vin1: value Conn_01x01_Male -> 5v
- Vin2: value Conn_01x01_Male -> 3v
- moved R2 3.81 mm to (158.8, 100.3)
- moved D2 2.84 mm to (238.8, 119.4)
- moved R3 1.27 mm to (167.6, 114.3)
Connections:
- D2 pad 2: Net-(1k2-Pad2) -> Net-(D2-Pad2)
Routing:
- net Net-(1k2-Pad2): track 257.0 -> 156.6 mm
- net Net-(R8-Pad1): track 49.7 -> 32.5 mm
- net Net-(D2-Pad2): track 0.00 -> 4.05 mm
- net Net-(R1-Pad1): track 16.1 -> 12.7 mm
- net Net-(C2-Pad1): track 38.6 -> 37.1 mm
- net Net-(R5-Pad1): track 18.2 -> 19.6 mm
- net Net-(R1-Pad2): track 6.53 -> 5.13 mm
- net Net-(C1-Pad1): track 26.7 -> 25.9 mm
- net Net-(1k2-Pad1): track 25.4 -> 26.1 mm
- net Net-(D1-Pad2): track 39.9 -> 39.3 mm
Other:
- board text added: "AUBREY TARMU"
- board text removed: "gnd"
