File: Lab8/kicad/kicad.sch (KiCad schematic (older format))
At the start: 7 parts, among them J4 TI_BOOSTER_40_J4

Commit message: added some stuff to my lab8
Parts:
- added 1k: R4, symbol pspice:R
- added 1k: R7, symbol pspice:R
- added C2: 97.3uf, symbol pspice:CAP
- added R5: 20k, symbol pspice:R
- added R6: 842k, symbol pspice:R
- added R8: 15k, symbol pspice:R
- added U?: TLC277, symbol Amplifier_Operational:TLC277
- C1: renamed from C?; value CAP -> 97.3uf
- R3: renamed from R?; value R -> 680k
- gave numbers to parts that had none: 2
Changed lines of the file:
@@
 $EndComp
 $Comp
-L pspice:R R?
+L pspice:R R1
 U 1 1 61854D18
 P 3400 2950
-F 0 "R?" H 3468 2996 50  0000 L CNN
+F 0 "R1" H 3468 2996 50  0000 L CNN
 F 1 "R" H 3468 2905 50  0000 L CNN
 F 2 "" H 3400 2950 50  0001 C CNN
@@
 	3800 2700 3800 2750
 $Comp
-L pspice:R R?
+L pspice:R R2
 U 1 1 61857F5A
 P 3800 3000
-F 0 "R?" H 3868 3046 50  0000 L CNN
+F 0 "R2" H 3868 3046 50  0000 L CNN
 F 1 "R" H 3868 2955 50  0000 L CNN
 F 2 "" H 3800 3000 50  0001 C CNN
@@
 $EndComp
 $Comp
-L pspice:CAP C?
+L pspice:CAP C1
 U 1 1 618587C9
 P 4050 3250
-F 0 "C?" V 3735 3250 50  0000 C CNN
-F 1 "CAP" V 3826 3250 50  0000 C CNN
+F 0 "C1" V 3735 3250 50  0000 C CNN
+F 1 "97.3uf" V 3826 3250 50  0000 C CNN
 F 2 "" H 4050 3250 50  0001 C CNN
 F 3 "~" H 4050 3250 50  0001 C CNN
@@
 $EndComp
 $Comp
-L pspice:R R?
+L pspice:R R3
 U 1 1 6185965A
 P 4300 3500
-F 0 "R?" H 4232 3454 50  0000 R CNN
-F 1 "R" H 4232 3545 50  0000 R CNN
+F 0 "R3" H 4232 3454 50  0000 R CNN
+F 1 "680k" H 4232 3545 50  0000 R CNN
 F 2 "" H 4300 3500 50  0001 C CNN
 F 3 "~" H 4300 3500 50  0001 C CNN
@@
 	1    0    0    -1
 $EndComp
+$Comp
+L pspice:R R5
+U 1 1 61878E1F
+P 5000 3750
+F 0 "R5" H 4932 3704 50  0000 R CNN
+F 1 "20k" H 4932 3795 50  0000 R CNN
+F 2 "" H 5000 3750 50  0001 C CNN
+F 3 "~" H 5000 3750 50  0001 C CNN
+	1    5000 3750
+	0    1    1    0
+$EndComp
+$Comp
+L pspice:R 1k
+U 1 1 6187932D
+P 4700 4100
+F 0 "1k" H 4632 4054 50  0000 R CNN
+F 1 "R4" H 4632 4145 50  0000 R CNN
+F 2 "" H 4700 4100 50  0001 C CNN
+F 3 "~" H 4700 4100 50  0001 C CNN
+	1    4700 4100
+	1    0    0    -1
+$EndComp
+Wire Bus Line
+	4750 3450 4700 3450
+Wire Bus Line
+	4700 3450 4700 3750
+Wire Bus Line
+	4700 3750 4750 3750
+Wire Bus Line
+	4700 3750 4700 3850
+Connection ~ 4700 3750
+$Comp
+L power:GND #PWR?
+U 1 1 6187C7DD
+P 4700 4350
+F 0 "#PWR?" H 4700 4100 50  0001 C CNN
+F 1 "GND" H 4705 4177 50  0000 C CNN
+F 2 "" H 4700 4350 50  0001 C CNN
+F 3 "" H 4700 4350 50  0001 C CNN
+	1    4700 4350
+	1    0    0    -1
+$EndComp
+Wire Bus Line
+	5250 3750 5350 3750
+Wire Bus Line
+	5350 3750 5350 3350
+Wire Bus Line
+	5350 3350 5500 3350
+$Comp
+L pspice:R R6
+U 1 1 6187D634
+P 5750 3350
+F 0 "R6" H 5682 3304 50  0000 R CNN
+F 1 "842k" H 5682 3395 50  0000 R CNN
+F 2 "" H 5750 3350 50  0001 C CNN
+F 3 "~" H 5750 3350 50  0001 C CNN
+	1    5750 3350
+	0    -1   -1   0
+$EndComp
+Wire Bus Line
+	6000 3350 6150 3350
+$Comp
+L Amplifier_Operational:TLC277 U?
+U 1 1 61881D6C
+P 6750 3450
+F 0 "U?" H 6750 3817 50  0000 C CNN
+F 1 "TLC277" H 6750 3726 50  0000 C CNN
+F 2 "" H 6750 3450 50  0001 C CNN
+F 3 "http://www.ti.com/lit/ds/symlink/tlc272.pdf" H 6750 3450 50  0001 C CNN
+	1    6750 3450
+	1    0    0    -1
+$EndComp
+$Comp
+L pspice:R R8
+U 1 1 61881D72
+P 6700 3850
+F 0 "R8" H 6632 3804 50  0000 R CNN
+F 1 "15k" H 6632 3895 50  0000 R CNN
+F 2 "" H 6700 3850 50  0001 C CNN
+F 3 "~" H 6700 3850 50  0001 C CNN
+	1    6700 3850
+	0    1    1    0
+$EndComp
+$Comp
+L pspice:R 1k
+U 1 1 61881D78
+P 6400 4200
+F 0 "1k" H 6332 4154 50  0000 R CNN
+F 1 "R7" H 6332 4245 50  0000 R CNN
+F 2 "" H 6400 4200 50  0001 C CNN
+F 3 "~" H 6400 4200 50  0001 C CNN
+	1    6400 4200
+	1    0    0    -1
+$EndComp
+Wire Bus Line
+	6450 3550 6400 3550
+Wire Bus Line
+	6400 3550 6400 3850
+Wire Bus Line
+	6400 3850 6450 3850
+Wire Bus Line
+	6400 3850 6400 3950
+Connection ~ 6400 3850
+$Comp
+L power:GND #PWR?
+U 1 1 61881D83
+P 6400 4450
+F 0 "#PWR?" H 6400 4200 50  0001 C CNN
+F 1 "GND" H 6405 4277 50  0000 C CNN
+F 2 "" H 6400 4450 50  0001 C CNN
+F 3 "" H 6400 4450 50  0001 C CNN
+	1    6400 4450
+	1    0    0    -1
+$EndComp
+Wire Bus Line
+	6950 3850 7050 3850
+Wire Bus Line
+	7050 3850 7050 3450
+Wire Bus Line
+	7050 3450 7200 3450
+Wire Bus Line
+	6150 3350 6150 3500
+Connection ~ 6150 3350
+Wire Bus Line
+	6150 3350 6450 3350
+$Comp
+L pspice:CAP C2
+U 1 1 61883FA3
+P 6150 3750
+F 0 "C2" V 5835 3750 50  0000 C CNN
+F 1 "97.3uf" V 5926 3750 50  0000 C CNN
+F 2 "" H 6150 3750 50  0001 C CNN
+F 3 "~" H 6150 3750 50  0001 C CNN
+	1    6150 3750
+	1    0    0    -1
+$EndComp
+$Comp
+L power:GND #PWR?
+U 1 1 61884CBC
+P 6150 4000
+F 0 "#PWR?" H 6150 3750 50  0001 C CNN
+F 1 "GND" H 6155 3827 50  0000 C CNN
+F 2 "" H 6150 4000 50  0001 C CNN
+F 3 "" H 6150 4000 50  0001 C CNN
+	1    6150 4000
+	1    0    0    -1
+$EndComp

Commit message: nearly done w/8
Parts:
- added D? (x2): DIODE, symbol pspice:DIODE
- added R9: 100, symbol pspice:R
Connections:
- net labels added: +3.3V
- net labels removed: VCC
Changed lines of the file:
@@
-$EndComp
-$Comp
-L power:VCC #PWR02
-U 1 1 5080AA9F
-P 9150 750
-F 0 "#PWR02" H 9150 600 50  0001 C CNN
-F 1 "VCC" H 9150 900 50  0000 C CNN
-F 2 "" H 9150 750 50  0000 C CNN
-F 3 "" H 9150 750 50  0000 C CNN
-	1    9150 750
-	1    0    0    -1
 $EndComp
 $Comp
 L boosterpack:Ti_Booster_40_J4 J4
 U 1 1 5080DC12
-P 8450 2400
-F 0 "J4" H 8400 3050 60  0000 C CNN
-F 1 "TI_BOOSTER_40_J4" H 8450 1750 60  0000 C CNN
-F 2 "Connector_PinHeader_2.54mm:PinHeader_1x10_P2.54mm_Vertical" V 8900 2400 60  0001 C CNN
-F 3 "" H 8450 2400 60  0001 C CNN
-	1    8450 2400
+P 9200 3400
+F 0 "J4" H 9150 4050 60  0000 C CNN
+F 1 "TI_BOOSTER_40_J4" H 9200 2750 60  0000 C CNN
+F 2 "Connector_PinHeader_2.54mm:PinHeader_1x10_P2.54mm_Vertical" V 9650 3400 60  0001 C CNN
+F 3 "" H 9200 3400 60  0001 C CNN
+	1    9200 3400
 	1    0    0    -1
 $EndComp
@@
 	1    0    0    -1
 $EndComp
+$Comp
+L pspice:R R9
+U 1 1 61885D58
+P 7450 3450
+F 0 "R9" H 7382 3404 50  0000 R CNN
+F 1 "100" H 7382 3495 50  0000 R CNN
+F 2 "" H 7450 3450 50  0001 C CNN
+F 3 "~" H 7450 3450 50  0001 C CNN
+	1    7450 3450
+	0    1    1    0
+$EndComp
+$Comp
+L pspice:DIODE D?
+U 1 1 6188CB8D
+P 7700 3650
+F 0 "D?" V 7654 3778 50  0000 L CNN
+F 1 "DIODE" V 7745 3778 50  0000 L CNN
+F 2 "" H 7700 3650 50  0001 C CNN
+F 3 "~" H 7700 3650 50  0001 C CNN
+	1    7700 3650
+	0    1    1    0
+$EndComp
+$Comp
+L power:GND #PWR?
+U 1 1 6188CB93
+P 7700 3850
+F 0 "#PWR?" H 7700 3600 50  0001 C CNN
+F 1 "GND" H 7705 3677 50  0000 C CNN
+F 2 "" H 7700 3850 50  0001 C CNN
+F 3 "" H 7700 3850 50  0001 C CNN
+	1    7700 3850
+	1    0    0    -1
+$EndComp
+$Comp
+L pspice:DIODE D?
+U 1 1 6188D84B
+P 7700 3250
+F 0 "D?" V 7654 3378 50  0000 L CNN
+F 1 "DIODE" V 7745 3378 50  0000 L CNN
+F 2 "" H 7700 3250 50  0001 C CNN
+F 3 "~" H 7700 3250 50  0001 C CNN
+	1    7700 3250
+	0    1    1    0
+$EndComp
+Connection ~ 7700 3450
+$Comp
+L power:+3.3V #PWR?
+U 1 1 6188FA63
+P 7700 3050
+F 0 "#PWR?" H 7700 2900 50  0001 C CNN
+F 1 "+3.3V" H 7715 3223 50  0000 C CNN
+F 2 "" H 7700 3050 50  0001 C CNN
+F 3 "" H 7700 3050 50  0001 C CNN
+	1    7700 3050
+	1    0    0    -1
+$EndComp
+Wire Bus Line
+	8100 3450 7700 3450
+Wire Bus Line
+	7700 3450 8400 3450
+Wire Bus Line
+	8400 3450 8400 3550
+Wire Bus Line
+	8400 3550 8600 3550
 $EndSCHEMATC

Commit message: nearly done w/ lab08
Parts:
- removed D?: DIODE, symbol pspice:DIODE
- removed J4: TI_BOOSTER_40_J4, Connector_PinHeader_2.54mm:PinHeader_1x10_P2.54mm_Vertical, symbol boosterpack:Ti_Booster_40_J4
- added OUT, Vin1, Vin2, gnd1: Conn_01x01_Male, Connector_PinHeader_2.54mm:PinHeader_1x01_P2.54mm_Horizontal, symbol Connector:Conn_01x01_Male
- added U1: OPB745, Connector_PinSocket_2.54mm:PinSocket_1x08_P2.54mm_Vertical, symbol OPB745:OPB745
- 1k2: renamed from 1k; footprint (none) -> Resistor_SMD:R_0201_0603Metric
- C1: footprint (none) -> Capacitor_SMD:CP_Elec_3x5.4
- C2: footprint (none) -> Capacitor_SMD:CP_Elec_4x3
- D1, D2: renamed from D?; footprint (none) -> Diode_SMD:D_0201_0603Metric
- R1: value R -> 82.5; footprint (none) -> Resistor_SMD:R_0201_0603Metric
- R2: value R -> 10k; footprint (none) -> Resistor_SMD:R_0201_0603Metric
- R3, R5, R6, R8, R9: footprint (none) -> Resistor_SMD:R_0201_0603Metric
- U2, U3: renamed from U?; footprint (none) -> TLC277CP:DIP794W45P254L959H508Q8
- r4: renamed from 1k; value R4 -> 1k; footprint (none) -> Resistor_SMD:R_0201_0603Metric
Connections:
- net labels removed: +3.3V, +5V
- wire segments 0 -> 37

Commit message: some kicad stuff
Parts:
- OUT1: renamed from OUT; footprint Connector_PinHeader_2.54mm:PinHeader_1x01_P2.54mm_Horizontal -> Connector_PinHeader_2.54mm:PinHeader_1x07_P2.54mm_Vertical_SMD_Pin1Left
- U1: footprint Connector_PinSocket_2.54mm:PinSocket_1x08_P2.54mm_Vertical -> Connector_PinHeader_2.54mm:PinHeader_1x04_P2.54mm_Vertical
- Vin1, Vin2: footprint Connector_PinHeader_2.54mm:PinHeader_1x01_P2.54mm_Horizontal -> Connector_PinHeader_2.54mm:PinHeader_1x08_P2.54mm_Vertical_SMD_Pin1Left
- gnd1: footprint Connector_PinHeader_2.54mm:PinHeader_1x01_P2.54mm_Horizontal -> Connector_PinHeader_2.54mm:PinHeader_1x07_P2.54mm_Vertical_SMD_Pin1Left
Changed lines of the file:
@@
-$EndComp
-$Comp
-L pspice:CAP C2
-U 1 1 61883FA3
-P 6150 3750
-F 0 "C2" V 5835 3750 50  0000 C CNN
-F 1 "97.3uf" V 5926 3750 50  0000 C CNN
-F 2 "Capacitor_SMD:CP_Elec_4x3" H 6150 3750 50  0001 C CNN
-F 3 "~" H 6150 3750 50  0001 C CNN
-	1    6150 3750
-	1    0    0    -1
 $EndComp
 $Comp
@@
 F 0 "Vin1" H 3308 2881 50  0000 C CNN
 F 1 "Conn_01x01_Male" H 3308 2790 50  0000 C CNN
-F 2 "Connector_PinHeader_2.54mm:PinHeader_1x01_P2.54mm_Horizontal" H 3200 2700 50  0001 C CNN
+F 2 "Connector_PinHeader_2.54mm:PinHeader_1x08_P2.54mm_Vertical_SMD_Pin1Left" H 3200 2700 50  0001 C CNN
 F 3 "~" H 3200 2700 50  0001 C CNN
 	1    3200 2700
@@
 F 0 "gnd1" V 5504 4462 50  0000 R CNN
 F 1 "Conn_01x01_Male" V 5413 4462 50  0000 R CNN
-F 2 "Connector_PinHeader_2.54mm:PinHeader_1x01_P2.54mm_Horizontal" H 5350 4550 50  0001 C CNN
+F 2 "Connector_PinHeader_2.54mm:PinHeader_1x07_P2.54mm_Vertical_SMD_Pin1Left" H 5350 4550 50  0001 C CNN
 F 3 "~" H 5350 4550 50  0001 C CNN
 	1    5350 4550
@@
 Wire Wire Line
 	6150 3350 6150 3500
-Connection ~ 6150 3350
-Wire Wire Line
-	6150 3350 6450 3350
-$Comp
-L Amplifier_Operational:TLC277 U3
-U 1 1 61881D6C
-P 6750 3450
-F 0 "U3" H 6750 3817 50  0000 C CNN
-F 1 "TLC277" H 6750 3726 50  0000 C CNN
-F 2 "TLC277CP:DIP794W45P254L959H508Q8" H 6750 3450 50  0001 C CNN
-F 3 "http://www.ti.com/lit/ds/symlink/tlc272.pdf" H 6750 3450 50  0001 C CNN
-	1    6750 3450
-	1    0    0    -1
-$EndComp
 Wire Wire Line
 	6950 3850 7100 3850
@@
 F 0 "U1" H 4028 2496 50  0000 L CNN
 F 1 "OPB745" H 4028 2405 50  0000 L CNN
-F 2 "Connector_PinSocket_2.54mm:PinSocket_1x08_P2.54mm_Vertical" H 2800 3350 50  0001 L CNN
+F 2 "Connector_PinHeader_2.54mm:PinHeader_1x04_P2.54mm_Vertical" H 2800 3350 50  0001 L CNN
 F 3 "https://upverter.com/datasheet/4f8d3d5f99316b04551580b4d6f54087dceae820.pdf" H 2800 3450 50  0001 L CNN
 F 4 "IC" H 2800 3550 50  0001 L CNN "category"
@@
 F 0 "Vin2" H 7608 3231 50  0000 C CNN
 F 1 "Conn_01x01_Male" H 7608 3140 50  0000 C CNN
-F 2 "Connector_PinHeader_2.54mm:PinHeader_1x01_P2.54mm_Horizontal" H 7500 3050 50  0001 C CNN
+F 2 "Connector_PinHeader_2.54mm:PinHeader_1x08_P2.54mm_Vertical_SMD_Pin1Left" H 7500 3050 50  0001 C CNN
 F 3 "~" H 7500 3050 50  0001 C CNN
 	1    7500 3050
@@
 	6400 3950 6400 3850
 Wire Wire Line
-	6400 3550 6450 3550
-Wire Wire Line
 	6450 3850 6400 3850
-Connection ~ 6400 3850
-Wire Wire Line
-	6400 3850 6400 3550
-$Comp
-L Connector:Conn_01x01_Male OUT
+$Comp
+L Connector:Conn_01x01_Male OUT1
 U 1 1 6193298D
 P 8850 3450
-F 0 "OUT" H 8958 3631 50  0000 C CNN
+F 0 "OUT1" H 8958 3631 50  0000 C CNN
 F 1 "Conn_01x01_Male" H 8958 3540 50  0000 C CNN
-F 2 "Connector_PinHeader_2.54mm:PinHeader_1x01_P2.54mm_Horizontal" H 8850 3450 50  0001 C CNN
+F 2 "Connector_PinHeader_2.54mm:PinHeader_1x07_P2.54mm_Vertical_SMD_Pin1Left" H 8850 3450 50  0001 C CNN
 F 3 "~" H 8850 3450 50  0001 C CNN
 	1    8850 3450
@@
 Wire Wire Line
 	7700 3450 8650 3450
+Connection ~ 6400 3850
+Connection ~ 6150 3350
+Wire Wire Line
+	6400 3850 6400 3550
+Wire Wire Line
+	6400 3550 6450 3550
+Wire Wire Line
+	6150 3350 6450 3350
+$Comp
+L pspice:CAP C2
+U 1 1 61883FA3
+P 6150 3750
+F 0 "C2" V 5835 3750 50  0000 C CNN
+F 1 "97.3uf" V 5926 3750 50  0000 C CNN
+F 2 "Capacitor_SMD:CP_Elec_4x3" H 6150 3750 50  0001 C CNN
+F 3 "~" H 6150 3750 50  0001 C CNN
+	1    6150 3750
+	1    0    0    -1
+$EndComp
+$Comp
+L Amplifier_Operational:TLC277 U3
+U 1 1 61881D6C
+P 6750 3450
+F 0 "U3" H 6750 3817 50  0000 C CNN
+F 1 "TLC277" H 6750 3726 50  0000 C CNN
+F 2 "TLC277CP:DIP794W45P254L959H508Q8" H 6750 3450 50  0001 C CNN
+F 3 "http://www.ti.com/lit/ds/symlink/tlc272.pdf" H 6750 3450 50  0001 C CNN
+	1    6750 3450
+	1    0    0    -1
+$EndComp
 $EndSCHEMATC

Commit message: near checkoff
Parts:
- removed U3: TLC277, TLC277CP:DIP794W45P254L959H508Q8, symbol Amplifier_Operational:TLC277
- added unit 2 of U2
- OUT1, gnd1: footprint Connector_PinHeader_2.54mm:PinHeader_1x07_P2.54mm_Vertical_SMD_Pin1Left -> Connector_PinHeader_2.54mm:PinHeader_1x01_P2.54mm_Horizontal
- U1: symbol OPB745:OPB745 -> kicad-rescue:OPB745-OPB745
- Vin1, Vin2: footprint Connector_PinHeader_2.54mm:PinHeader_1x08_P2.54mm_Vertical_SMD_Pin1Left -> Connector_PinHeader_2.54mm:PinHeader_1x01_P2.54mm_Horizontal
Changed lines of the file:
@@
 F 0 "Vin1" H 3308 2881 50  0000 C CNN
 F 1 "Conn_01x01_Male" H 3308 2790 50  0000 C CNN
-F 2 "Connector_PinHeader_2.54mm:PinHeader_1x08_P2.54mm_Vertical_SMD_Pin1Left" H 3200 2700 50  0001 C CNN
+F 2 "Connector_PinHeader_2.54mm:PinHeader_1x01_P2.54mm_Horizontal" H 3200 2700 50  0001 C CNN
 F 3 "~" H 3200 2700 50  0001 C CNN
 	1    3200 2700
@@
 F 0 "gnd1" V 5504 4462 50  0000 R CNN
 F 1 "Conn_01x01_Male" V 5413 4462 50  0000 R CNN
-F 2 "Connector_PinHeader_2.54mm:PinHeader_1x07_P2.54mm_Vertical_SMD_Pin1Left" H 5350 4550 50  0001 C CNN
+F 2 "Connector_PinHeader_2.54mm:PinHeader_1x01_P2.54mm_Horizontal" H 5350 4550 50  0001 C CNN
 F 3 "~" H 5350 4550 50  0001 C CNN
 	1    5350 4550
@@
 Connection ~ 3800 3250
 $Comp
-L OPB745:OPB745 U1
+L kicad-rescue:OPB745-OPB745 U1
 U 1 1 61872E79
 P 2800 3150
@@
 F 0 "Vin2" H 7608 3231 50  0000 C CNN
 F 1 "Conn_01x01_Male" H 7608 3140 50  0000 C CNN
-F 2 "Connector_PinHeader_2.54mm:PinHeader_1x08_P2.54mm_Vertical_SMD_Pin1Left" H 7500 3050 50  0001 C CNN
+F 2 "Connector_PinHeader_2.54mm:PinHeader_1x01_P2.54mm_Horizontal" H 7500 3050 50  0001 C CNN
 F 3 "~" H 7500 3050 50  0001 C CNN
 	1    7500 3050
@@
 F 0 "OUT1" H 8958 3631 50  0000 C CNN
 F 1 "Conn_01x01_Male" H 8958 3540 50  0000 C CNN
-F 2 "Connector_PinHeader_2.54mm:PinHeader_1x07_P2.54mm_Vertical_SMD_Pin1Left" H 8850 3450 50  0001 C CNN
+F 2 "Connector_PinHeader_2.54mm:PinHeader_1x01_P2.54mm_Horizontal" H 8850 3450 50  0001 C CNN
 F 3 "~" H 8850 3450 50  0001 C CNN
 	1    8850 3450
@@
 $EndComp
 $Comp
-L Amplifier_Operational:TLC277 U3
-U 1 1 61881D6C
+L Amplifier_Operational:TLC277 U2
+U 2 1 6188DFF6
 P 6750 3450
-F 0 "U3" H 6750 3817 50  0000 C CNN
+F 0 "U2" H 6750 3817 50  0000 C CNN
 F 1 "TLC277" H 6750 3726 50  0000 C CNN
 F 2 "TLC277CP:DIP794W45P254L959H508Q8" H 6750 3450 50  0001 C CNN
 F 3 "http://www.ti.com/lit/ds/symlink/tlc272.pdf" H 6750 3450 50  0001 C CNN
-	1    6750 3450
-	1    0    0    -1
-$EndComp
+	2    6750 3450
+	1    0    0    -1
+$EndComp

Commit message: fixed the clearance issue
Parts:
- R1, R2, R3, R5, R6, R8, R9, r4: footprint Resistor_SMD:R_0201_0603Metric -> Resistor_SMD:R_0201_0603Metric_Pad0.64x0.40mm_HandSolder
Changed lines of the file:
@@
 F 0 "R1" H 3468 2996 50  0000 L CNN
 F 1 "82.5" H 3468 2905 50  0000 L CNN
-F 2 "Resistor_SMD:R_0201_0603Metric" H 3400 2950 50  0001 C CNN
+F 2 "Resistor_SMD:R_0201_0603Metric_Pad0.64x0.40mm_HandSolder" H 3400 2950 50  0001 C CNN
 F 3 "~" H 3400 2950 50  0001 C CNN
 	1    3400 2950
@@
 F 0 "R2" H 3868 3046 50  0000 L CNN
 F 1 "10k" H 3868 2955 50  0000 L CNN
-F 2 "Resistor_SMD:R_0201_0603Metric" H 3800 3000 50  0001 C CNN
+F 2 "Resistor_SMD:R_0201_0603Metric_Pad0.64x0.40mm_HandSolder" H 3800 3000 50  0001 C CNN
 F 3 "~" H 3800 3000 50  0001 C CNN
 	1    3800 3000
@@
 F 0 "R3" H 4232 3454 50  0000 R CNN
 F 1 "680k" H 4232 3545 50  0000 R CNN
-F 2 "Resistor_SMD:R_0201_0603Metric" H 4300 3500 50  0001 C CNN
+F 2 "Resistor_SMD:R_0201_0603Metric_Pad0.64x0.40mm_HandSolder" H 4300 3500 50  0001 C CNN
 F 3 "~" H 4300 3500 50  0001 C CNN
 	1    4300 3500
@@
 F 0 "r4" H 4632 4054 50  0000 R CNN
 F 1 "1k" H 4632 4145 50  0000 R CNN
-F 2 "Resistor_SMD:R_0201_0603Metric" H 4700 4100 50  0001 C CNN
+F 2 "Resistor_SMD:R_0201_0603Metric_Pad0.64x0.40mm_HandSolder" H 4700 4100 50  0001 C CNN
 F 3 "~" H 4700 4100 50  0001 C CNN
 	1    4700 4100
@@
 F 0 "R6" H 5682 3304 50  0000 R CNN
 F 1 "842k" H 5682 3395 50  0000 R CNN
-F 2 "Resistor_SMD:R_0201_0603Metric" H 5750 3350 50  0001 C CNN
+F 2 "Resistor_SMD:R_0201_0603Metric_Pad0.64x0.40mm_HandSolder" H 5750 3350 50  0001 C CNN
 F 3 "~" H 5750 3350 50  0001 C CNN
 	1    5750 3350
@@
 F 0 "R9" H 7382 3404 50  0000 R CNN
 F 1 "100" H 7382 3495 50  0000 R CNN
-F 2 "Resistor_SMD:R_0201_0603Metric" H 7450 3450 50  0001 C CNN
+F 2 "Resistor_SMD:R_0201_0603Metric_Pad0.64x0.40mm_HandSolder" H 7450 3450 50  0001 C CNN
 F 3 "~" H 7450 3450 50  0001 C CNN
 	1    7450 3450
@@
 F 0 "R5" H 4932 3704 50  0000 R CNN
 F 1 "20k" H 4932 3795 50  0000 R CNN
-F 2 "Resistor_SMD:R_0201_0603Metric" H 5000 3750 50  0001 C CNN
+F 2 "Resistor_SMD:R_0201_0603Metric_Pad0.64x0.40mm_HandSolder" H 5000 3750 50  0001 C CNN
 F 3 "~" H 5000 3750 50  0001 C CNN
 	1    5000 3750
@@
 F 0 "R8" H 6632 3804 50  0000 R CNN
 F 1 "15k" H 6632 3895 50  0000 R CNN
-F 2 "Resistor_SMD:R_0201_0603Metric" H 6700 3850 50  0001 C CNN
+F 2 "Resistor_SMD:R_0201_0603Metric_Pad0.64x0.40mm_HandSolder" H 6700 3850 50  0001 C CNN
 F 3 "~" H 6700 3850 50  0001 C CNN
 	1    6700 3850
