File: Lab8/kicad/kicad.sch (KiCad schematic (older format))
At the start: 19 parts, among them U1 OPB745, U2 TLC277

Commit message: pcb done
Parts:
- U1: Spice_Model (none) -> dc 1 ac 1; Spice_Netlist_Enabled (none) -> Y; Spice_Primitive (none) -> I
Other:
- note added: "Aubrey Tarmu\n11-12-21\n"
- note added: "Heart Rate Monitor\n"
Changed lines of the file:
@@
 $EndDescr
-$Comp
-L power:GND #PWR01
-U 1 1 5080AA99
-P 11450 2300
-F 0 "#PWR01" H 11450 2050 50  0001 C CNN
-F 1 "GND" H 11450 2150 50  0000 C CNN
-F 2 "" H 11450 2300 50  0000 C CNN
-F 3 "" H 11450 2300 50  0000 C CNN
-	1    11450 2300
-	0    1    1    0
-$EndComp
 $Comp
 L pspice:R R1
@@
 	1    3800 3000
 	1    0    0    -1
-$EndComp
-$Comp
-L pspice:CAP C1
-U 1 1 618587C9
-P 4050 3250
-F 0 "C1" V 3735 3250 50  0000 C CNN
-F 1 "97.3uf" V 3826 3250 50  0000 C CNN
-F 2 "Capacitor_SMD:CP_Elec_3x5.4" H 4050 3250 50  0001 C CNN
-F 3 "~" H 4050 3250 50  0001 C CNN
-	1    4050 3250
-	0    1    1    0
 $EndComp
 $Comp
@@
 $EndComp
 Connection ~ 5350 3350
+Wire Wire Line
+	4700 3850 4700 3750
+Wire Wire Line
+	4700 3450 4750 3450
+Wire Wire Line
+	4750 3750 4700 3750
+Connection ~ 4700 3750
+Wire Wire Line
+	4700 3750 4700 3450
+Wire Wire Line
+	4750 3250 4300 3250
+Connection ~ 4300 3250
+Wire Wire Line
+	3400 2700 3800 2700
+Wire Wire Line
+	3800 2700 3800 2750
+Connection ~ 3400 2700
+Wire Wire Line
+	3400 3250 3400 3200
+Wire Wire Line
+	3400 3250 2800 3250
+Connection ~ 7700 3450
+$Comp
+L pspice:DIODE D2
+U 1 1 6188CB8D
+P 7700 3650
+F 0 "D2" V 7654 3778 50  0000 L CNN
+F 1 "DIODE" V 7745 3778 50  0000 L CNN
+F 2 "Diode_SMD:D_0201_0603Metric" H 7700 3650 50  0001 C CNN
+F 3 "~" H 7700 3650 50  0001 C CNN
+	1    7700 3650
+	0    1    1    0
+$EndComp
+$Comp
+L Connector:Conn_01x01_Male Vin2
+U 1 1 618E2A83
+P 7500 3050
+F 0 "Vin2" H 7608 3231 50  0000 C CNN
+F 1 "Conn_01x01_Male" H 7608 3140 50  0000 C CNN
+F 2 "Connector_PinHeader_2.54mm:PinHeader_1x01_P2.54mm_Horizontal" H 7500 3050 50  0001 C CNN
+F 3 "~" H 7500 3050 50  0001 C CNN
+	1    7500 3050
+	1    0    0    -1
+$EndComp
+Wire Wire Line
+	7700 3850 7700 4450
+Wire Wire Line
+	7700 4450 6400 4450
+Wire Wire Line
+	4700 4350 5350 4350
+Wire Wire Line
+	6100 4350 6100 4450
+Wire Wire Line
+	6100 4450 6150 4450
+Connection ~ 6400 4450
+Wire Wire Line
+	4700 4450 4700 4350
+Connection ~ 4700 4350
+Connection ~ 5350 4350
+Wire Wire Line
+	5350 4350 6100 4350
+Wire Wire Line
+	6150 4000 6150 4450
+Connection ~ 6150 4450
+Wire Wire Line
+	6150 4450 6400 4450
+Wire Wire Line
+	4300 3750 4300 4450
+Connection ~ 4300 4450
+Wire Wire Line
+	4300 4450 4700 4450
+$Comp
+L pspice:R R8
+U 1 1 61881D72
+P 6700 3850
+F 0 "R8" H 6632 3804 50  0000 R CNN
+F 1 "15k" H 6632 3895 50  0000 R CNN
+F 2 "Resistor_SMD:R_0201_0603Metric_Pad0.64x0.40mm_HandSolder" H 6700 3850 50  0001 C CNN
+F 3 "~" H 6700 3850 50  0001 C CNN
+	1    6700 3850
+	0    1    1    0
+$EndComp
+Wire Wire Line
+	6400 3950 6400 3850
+Wire Wire Line
+	6450 3850 6400 3850
+$Comp
+L Connector:Conn_01x01_Male OUT1
+U 1 1 6193298D
+P 8850 3450
+F 0 "OUT1" H 8958 3631 50  0000 C CNN
+F 1 "Conn_01x01_Male" H 8958 3540 50  0000 C CNN
+F 2 "Connector_PinHeader_2.54mm:PinHeader_1x01_P2.54mm_Horizontal" H 8850 3450 50  0001 C CNN
+F 3 "~" H 8850 3450 50  0001 C CNN
+	1    8850 3450
+	-1   0    0    1
+$EndComp
+Wire Wire Line
+	7700 3450 8650 3450
+Connection ~ 6400 3850
+Connection ~ 6150 3350
+Wire Wire Line
+	6400 3850 6400 3550
+Wire Wire Line
+	6400 3550 6450 3550
+Wire Wire Line
+	6150 3350 6450 3350
+$Comp
+L pspice:CAP C2
+U 1 1 61883FA3
+P 6150 3750
+F 0 "C2" V 5835 3750 50  0000 C CNN
+F 1 "97.3uf" V 5926 3750 50  0000 C CNN
+F 2 "Capacitor_SMD:CP_Elec_4x3" H 6150 3750 50  0001 C CNN
+F 3 "~" H 6150 3750 50  0001 C CNN
+	1    6150 3750
+	1    0    0    -1
+$EndComp
+$Comp
+L Amplifier_Operational:TLC277 U2
+U 2 1 6188DFF6
+P 6750 3450
+F 0 "U2" H 6750 3817 50  0000 C CNN
+F 1 "TLC277" H 6750 3726 50  0000 C CNN
+F 2 "TLC277CP:DIP794W45P254L959H508Q8" H 6750 3450 50  0001 C CNN
+F 3 "http://www.ti.com/lit/ds/symlink/tlc272.pdf" H 6750 3450 50  0001 C CNN
+	2    6750 3450
+	1    0    0    -1
+$EndComp
+$Comp
+L pspice:CAP C1
+U 1 1 618587C9
+P 4050 3250
+F 0 "C1" V 3735 3250 50  0000 C CNN
+F 1 "97.3uf" V 3826 3250 50  0000 C CNN
+F 2 "Capacitor_SMD:CP_Elec_3x5.4" H 4050 3250 50  0001 C CNN
+F 3 "~" H 4050 3250 50  0001 C CNN
+	1    4050 3250
+	0    1    1    0
+$EndComp
 $Comp
 L Amplifier_Operational:TLC277 U2
@@
 	1    0    0    -1
 $EndComp
-Wire Wire Line
-	4700 3850 4700 3750
-Wire Wire Line
-	4700 3450 4750 3450
-Wire Wire Line
-	4750 3750 4700 3750
-Connection ~ 4700 3750
-Wire Wire Line
-	4700 3750 4700 3450
-Wire Wire Line
-	4750 3250 4300 3250
-Connection ~ 4300 3250
-Wire Wire Line
-	3400 2700 3800 2700
-Wire Wire Line
-	3800 2700 3800 2750
-Connection ~ 3400 2700
-Wire Wire Line
-	3400 3250 3400 3200
-Wire Wire Line
-	3400 3250 2800 3250
 Connection ~ 3800 3250
+Wire Wire Line
+	3800 4450 2800 4450
+Wire Wire Line
+	3800 4450 4300 4450
+Connection ~ 3800 4450
 $Comp
 L kicad-rescue:OPB745-OPB745 U1
@@
 F 14 "-40°C" H 2800 4550 50  0001 L CNN "temperature range low"
 F 15 "15V" H 2800 4650 50  0001 L CNN "voltage"
+F 16 "I" H 2800 3150 50  0001 C CNN "Spice_Primitive"
+F 17 "dc 1 ac 1" H 2800 3150 50  0001 C CNN "Spice_Model"
+F 18 "Y" H 2800 3150 50  0001 C CNN "Spice_Netlist_Enabled"
 	1    2800 3150
 	1    0    0    -1
 $EndComp
-Wire Wire Line
-	3800 4450 2800 4450
-Connection ~ 7700 3450
-$Comp
-L pspice:DIODE D2
-U 1 1 6188CB8D
-P 7700 3650
-F 0 "D2" V 7654 3778 50  0000 L CNN
-F 1 "DIODE" V 7745 3778 50  0000 L CNN
-F 2 "Diode_SMD:D_0201_0603Metric" H 7700 3650 50  0001 C CNN
-F 3 "~" H 7700 3650 50  0001 C CNN
-	1    7700 3650
-	0    1    1    0
-$EndComp
-$Comp
-L Connector:Conn_01x01_Male Vin2
-U 1 1 618E2A83
-P 7500 3050
-F 0 "Vin2" H 7608 3231 50  0000 C CNN
-F 1 "Conn_01x01_Male" H 7608 3140 50  0000 C CNN
-F 2 "Connector_PinHeader_2.54mm:PinHeader_1x01_P2.54mm_Horizontal" H 7500 3050 50  0001 C CNN
-F 3 "~" H 7500 3050 50  0001 C CNN
-	1    7500 3050
-	1    0    0    -1
-$EndComp
-Wire Wire Line
-	7700 3850 7700 4450
-Wire Wire Line
-	7700 4450 6400 4450
-Wire Wire Line
-	4700 4350 5350 4350
-Wire Wire Line
-	6100 4350 6100 4450
-Wire Wire Line
-	6100 4450 6150 4450
-Connection ~ 6400 4450
-Wire Wire Line
-	3800 4450 4300 4450
-Wire Wire Line
-	4700 4450 4700 4350
-Connection ~ 3800 4450
-Connection ~ 4700 4350
-Connection ~ 5350 4350
-Wire Wire Line
-	5350 4350 6100 4350
-Wire Wire Line
-	6150 4000 6150 4450
-Connection ~ 6150 4450
-Wire Wire Line
-	6150 4450 6400 4450
-Wire Wire Line
-	4300 3750 4300 4450
-Connection ~ 4300 4450
-Wire Wire Line
-	4300 4450 4700 4450
-$Comp
-L pspice:R R8
-U 1 1 61881D72
-P 6700 3850
-F 0 "R8" H 6632 3804 50  0000 R CNN
-F 1 "15k" H 6632 3895 50  0000 R CNN
-F 2 "Resistor_SMD:R_0201_0603Metric_Pad0.64x0.40mm_HandSolder" H 6700 3850 50  0001 C CNN
-F 3 "~" H 6700 3850 50  0001 C CNN
-	1    6700 3850
-	0    1    1    0
-$EndComp
-Wire Wire Line
-	6400 3950 6400 3850
-Wire Wire Line
-	6450 3850 6400 3850
-$Comp
-L Connector:Conn_01x01_Male OUT1
-U 1 1 6193298D
-P 8850 3450
-F 0 "OUT1" H 8958 3631 50  0000 C CNN
-F 1 "Conn_01x01_Male" H 8958 3540 50  0000 C CNN
-F 2 "Connector_PinHeader_2.54mm:PinHeader_1x01_P2.54mm_Horizontal" H 8850 3450 50  0001 C CNN
-F 3 "~" H 8850 3450 50  0001 C CNN
-	1    8850 3450
-	-1   0    0    1
-$EndComp
-Wire Wire Line
-	7700 3450 8650 3450
-Connection ~ 6400 3850
-Connection ~ 6150 3350
-Wire Wire Line
-	6400 3850 6400 3550
-Wire Wire Line
-	6400 3550 6450 3550
-Wire Wire Line
-	6150 3350 6450 3350
-$Comp
-L pspice:CAP C2
-U 1 1 61883FA3
-P 6150 3750
-F 0 "C2" V 5835 3750 50  0000 C CNN
-F 1 "97.3uf" V 5926 3750 50  0000 C CNN
-F 2 "Capacitor_SMD:CP_Elec_4x3" H 6150 3750 50  0001 C CNN
-F 3 "~" H 6150 3750 50  0001 C CNN
-	1    6150 3750
-	1    0    0    -1
-$EndComp
-$Comp
-L Amplifier_Operational:TLC277 U2
-U 2 1 6188DFF6
-P 6750 3450
-F 0 "U2" H 6750 3817 50  0000 C CNN
-F 1 "TLC277" H 6750 3726 50  0000 C CNN
-F 2 "TLC277CP:DIP794W45P254L959H508Q8" H 6750 3450 50  0001 C CNN
-F 3 "http://www.ti.com/lit/ds/symlink/tlc272.pdf" H 6750 3450 50  0001 C CNN
-	2    6750 3450
-	1    0    0    -1
-$EndComp
+Text Notes 8100 7500 2    50   ~ 0
+Heart Rate Monitor\n
+Text Notes 7550 6800 2    50   ~ 0
+Aubrey Tarmu\n11-12-21\n
 $EndSCHEMATC
