File: Lab8/kicad/kicad.sch (KiCad schematic (older format))
At the start: 19 parts, among them U1 OPB745, U2 TLC277

Commit message: fixed some stuff
Parts:
- added GND2: GND, Connector_PinHeader_2.54mm:PinHeader_1x01_P2.54mm_Horizontal, symbol Connector:Conn_01x01_Male
- 1k2, R1, R2, R3, R5, R6, R8, R9, r4: footprint Resistor_SMD:R_0201_0603Metric -> Resistor_THT:R_Axial_DIN0204_L3.6mm_D1.6mm_P1.90mm_Vertical
- C1: footprint Capacitor_SMD:CP_Elec_3x5.4 -> Capacitor_THT:CP_Radial_D4.0mm_P1.50mm
- C2: footprint Capacitor_SMD:CP_Elec_4x3 -> Capacitor_THT:CP_Radial_D4.0mm_P1.50mm
- D1, D2: footprint Diode_SMD:D_0201_0603Metric -> Capacitor_THT:CP_Axial_L10.0mm_D4.5mm_P15.00mm_Horizontal
- GND1: renamed from gnd1; value Conn_01x01_Male -> GND
- Vin1: value Conn_01x01_Male -> 5v
- Vin2: value Conn_01x01_Male -> 3v
Connections:
- net at 1k2.2, C2.2, GND1.1 (Pin_1)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: no longer D2.2 (A)
- new net: D2.2 (A), GND2.1 (Pin_1)
Changed lines of the file:
@@
 $EndDescr
-$Comp
-L power:GND #PWR01
-U 1 1 5080AA99
-P 11450 2300
-F 0 "#PWR01" H 11450 2050 50  0001 C CNN
-F 1 "GND" H 11450 2150 50  0000 C CNN
-F 2 "" H 11450 2300 50  0000 C CNN
-F 3 "" H 11450 2300 50  0000 C CNN
-	1    11450 2300
-	0    1    1    0
-$EndComp
 $Comp
 L pspice:R R1
@@
 F 0 "R1" H 3468 2996 50  0000 L CNN
 F 1 "82.5" H 3468 2905 50  0000 L CNN
-F 2 "Resistor_SMD:R_0201_0603Metric" H 3400 2950 50  0001 C CNN
+F 2 "Resistor_THT:R_Axial_DIN0204_L3.6mm_D1.6mm_P1.90mm_Vertical" H 3400 2950 50  0001 C CNN
 F 3 "~" H 3400 2950 50  0001 C CNN
 	1    3400 2950
@@
 F 0 "R2" H 3868 3046 50  0000 L CNN
 F 1 "10k" H 3868 2955 50  0000 L CNN
-F 2 "Resistor_SMD:R_0201_0603Metric" H 3800 3000 50  0001 C CNN
+F 2 "Resistor_THT:R_Axial_DIN0204_L3.6mm_D1.6mm_P1.90mm_Vertical" H 3800 3000 50  0001 C CNN
 F 3 "~" H 3800 3000 50  0001 C CNN
 	1    3800 3000
@@
 F 0 "C1" V 3735 3250 50  0000 C CNN
 F 1 "97.3uf" V 3826 3250 50  0000 C CNN
-F 2 "Capacitor_SMD:CP_Elec_3x5.4" H 4050 3250 50  0001 C CNN
+F 2 "Capacitor_THT:CP_Radial_D4.0mm_P1.50mm" H 4050 3250 50  0001 C CNN
 F 3 "~" H 4050 3250 50  0001 C CNN
 	1    4050 3250
@@
 F 0 "R3" H 4232 3454 50  0000 R CNN
 F 1 "680k" H 4232 3545 50  0000 R CNN
-F 2 "Resistor_SMD:R_0201_0603Metric" H 4300 3500 50  0001 C CNN
+F 2 "Resistor_THT:R_Axial_DIN0204_L3.6mm_D1.6mm_P1.90mm_Vertical" H 4300 3500 50  0001 C CNN
 F 3 "~" H 4300 3500 50  0001 C CNN
 	1    4300 3500
@@
 F 0 "r4" H 4632 4054 50  0000 R CNN
 F 1 "1k" H 4632 4145 50  0000 R CNN
-F 2 "Resistor_SMD:R_0201_0603Metric" H 4700 4100 50  0001 C CNN
+F 2 "Resistor_THT:R_Axial_DIN0204_L3.6mm_D1.6mm_P1.90mm_Vertical" H 4700 4100 50  0001 C CNN
 F 3 "~" H 4700 4100 50  0001 C CNN
 	1    4700 4100
@@
 F 0 "R6" H 5682 3304 50  0000 R CNN
 F 1 "842k" H 5682 3395 50  0000 R CNN
-F 2 "Resistor_SMD:R_0201_0603Metric" H 5750 3350 50  0001 C CNN
+F 2 "Resistor_THT:R_Axial_DIN0204_L3.6mm_D1.6mm_P1.90mm_Vertical" H 5750 3350 50  0001 C CNN
 F 3 "~" H 5750 3350 50  0001 C CNN
 	1    5750 3350
@@
 F 0 "R9" H 7382 3404 50  0000 R CNN
 F 1 "100" H 7382 3495 50  0000 R CNN
-F 2 "Resistor_SMD:R_0201_0603Metric" H 7450 3450 50  0001 C CNN
+F 2 "Resistor_THT:R_Axial_DIN0204_L3.6mm_D1.6mm_P1.90mm_Vertical" H 7450 3450 50  0001 C CNN
 F 3 "~" H 7450 3450 50  0001 C CNN
 	1    7450 3450
@@
 F 0 "D1" V 7654 3378 50  0000 L CNN
 F 1 "DIODE" V 7745 3378 50  0000 L CNN
-F 2 "Diode_SMD:D_0201_0603Metric" H 7700 3250 50  0001 C CNN
+F 2 "Capacitor_THT:CP_Axial_L10.0mm_D4.5mm_P15.00mm_Horizontal" H 7700 3250 50  0001 C CNN
 F 3 "~" H 7700 3250 50  0001 C CNN
 	1    7700 3250
@@
 F 0 "1k2" H 6332 4154 50  0000 R CNN
 F 1 "R7" H 6332 4245 50  0000 R CNN
-F 2 "Resistor_SMD:R_0201_0603Metric" H 6400 4200 50  0001 C CNN
+F 2 "Resistor_THT:R_Axial_DIN0204_L3.6mm_D1.6mm_P1.90mm_Vertical" H 6400 4200 50  0001 C CNN
 F 3 "~" H 6400 4200 50  0001 C CNN
 	1    6400 4200
@@
 P 3200 2700
 F 0 "Vin1" H 3308 2881 50  0000 C CNN
-F 1 "Conn_01x01_Male" H 3308 2790 50  0000 C CNN
+F 1 "5v" H 3308 2790 50  0000 C CNN
 F 2 "Connector_PinHeader_2.54mm:PinHeader_1x01_P2.54mm_Horizontal" H 3200 2700 50  0001 C CNN
 F 3 "~" H 3200 2700 50  0001 C CNN
@@
 $EndComp
 $Comp
-L Connector:Conn_01x01_Male gnd1
+L Connector:Conn_01x01_Male GND1
 U 1 1 6188AA28
 P 5350 4550
-F 0 "gnd1" V 5504 4462 50  0000 R CNN
-F 1 "Conn_01x01_Male" V 5413 4462 50  0000 R CNN
+F 0 "GND1" V 5504 4462 50  0000 R CNN
+F 1 "GND" V 5413 4462 50  0000 R CNN
 F 2 "Connector_PinHeader_2.54mm:PinHeader_1x01_P2.54mm_Horizontal" H 5350 4550 50  0001 C CNN
 F 3 "~" H 5350 4550 50  0001 C CNN
@@
 F 0 "R5" H 4932 3704 50  0000 R CNN
 F 1 "20k" H 4932 3795 50  0000 R CNN
-F 2 "Resistor_SMD:R_0201_0603Metric" H 5000 3750 50  0001 C CNN
+F 2 "Resistor_THT:R_Axial_DIN0204_L3.6mm_D1.6mm_P1.90mm_Vertical" H 5000 3750 50  0001 C CNN
 F 3 "~" H 5000 3750 50  0001 C CNN
 	1    5000 3750
@@
 F 0 "D2" V 7654 3778 50  0000 L CNN
 F 1 "DIODE" V 7745 3778 50  0000 L CNN
-F 2 "Diode_SMD:D_0201_0603Metric" H 7700 3650 50  0001 C CNN
+F 2 "Capacitor_THT:CP_Axial_L10.0mm_D4.5mm_P15.00mm_Horizontal" H 7700 3650 50  0001 C CNN
 F 3 "~" H 7700 3650 50  0001 C CNN
 	1    7700 3650
@@
 P 7500 3050
 F 0 "Vin2" H 7608 3231 50  0000 C CNN
-F 1 "Conn_01x01_Male" H 7608 3140 50  0000 C CNN
+F 1 "3v" H 7608 3140 50  0000 C CNN
 F 2 "Connector_PinHeader_2.54mm:PinHeader_1x01_P2.54mm_Horizontal" H 7500 3050 50  0001 C CNN
 F 3 "~" H 7500 3050 50  0001 C CNN
@@
 	7700 3850 7700 4450
 Wire Wire Line
-	7700 4450 6400 4450
-Wire Wire Line
 	4700 4350 5350 4350
 Wire Wire Line
@@
 Wire Wire Line
 	6100 4450 6150 4450
-Connection ~ 6400 4450
 Wire Wire Line
 	3800 4450 4300 4450
@@
 F 0 "R8" H 6632 3804 50  0000 R CNN
 F 1 "15k" H 6632 3895 50  0000 R CNN
-F 2 "Resistor_SMD:R_0201_0603Metric" H 6700 3850 50  0001 C CNN
+F 2 "Resistor_THT:R_Axial_DIN0204_L3.6mm_D1.6mm_P1.90mm_Vertical" H 6700 3850 50  0001 C CNN
 F 3 "~" H 6700 3850 50  0001 C CNN
 	1    6700 3850
@@
 F 0 "C2" V 5835 3750 50  0000 C CNN
 F 1 "97.3uf" V 5926 3750 50  0000 C CNN
-F 2 "Capacitor_SMD:CP_Elec_4x3" H 6150 3750 50  0001 C CNN
+F 2 "Capacitor_THT:CP_Radial_D4.0mm_P1.50mm" H 6150 3750 50  0001 C CNN
 F 3 "~" H 6150 3750 50  0001 C CNN
 	1    6150 3750
@@
 	1    0    0    -1
 $EndComp
+$Comp
+L Connector:Conn_01x01_Male GND2
+U 1 1 61935FB2
+P 7700 4650
+F 0 "GND2" V 7854 4562 50  0000 R CNN
+F 1 "GND" V 7763 4562 50  0000 R CNN
+F 2 "Connector_PinHeader_2.54mm:PinHeader_1x01_P2.54mm_Horizontal" H 7700 4650 50  0001 C CNN
+F 3 "~" H 7700 4650 50  0001 C CNN
+	1    7700 4650
+	0    -1   -1   0
+$EndComp
 $EndSCHEMATC
